Commit message: changes

File: clearpath_platform_description/urdf/a200/wheels/wheel.urdf.xacro (robot description, xacro)
@@ -1,15 +1,15 @@
 <?xml version="1.0"?>
-<robot xmlns:xacro="http://ros.org/wiki/xacro" name="wheel">
-  <xacro:macro name="wheel" params="wheel_prefix *joint_pose">
+<robot xmlns:xacro="http://ros.org/wiki/xacro" name="a200_wheel">
+  <xacro:macro name="a200_wheel" params="wheel_prefix *joint_pose">
     <link name="${wheel_prefix}_wheel">
       <inertial>
         <mass value="2.637" />
         <origin xyz="0 0 0" />
-        <inertia  ixx="0.02467" ixy="0" ixz="0" iyy="0.04411" iyz="0" izz="0.02467" />
+        <inertia ixx="0.02467" ixy="0" ixz="0" iyy="0.04411" iyz="0" izz="0.02467" />
       </inertial>
       <visual>
         <origin xyz="0 0 0" rpy="0 0 0" />
         <geometry>
-          <mesh filename="package://clearpath_platform_description/meshes/wheel.dae" />
+          <mesh filename="package://clearpath_platform_description/meshes/a200/wheel.dae" />
         </geometry>
       </visual>
@@ -21,11 +21,11 @@
       </collision>
     </link>
-    <gazebo reference="${wheel_prefix}_wheel">
+    <!-- <gazebo reference="${wheel_prefix}_wheel">
       <mu1 value="1.0"/>
       <mu2 value="0.5"/>
-      <kp value="10000000.0" />
+      <kp value="100000000000000000000.0" />
       <kd value="1.0" />
       <fdir1 value="1 0 0"/>
-    </gazebo>
+    </gazebo> -->
     <joint name="${wheel_prefix}_wheel_joint" type="continuous">
       <parent link="base_link"/>

File: clearpath_platform_description/urdf/husky.urdf.xacro (robot description, xacro)
@@ -1,11 +1,9 @@
 <?xml version="1.0"?>
 <robot xmlns:xacro="http://ros.org/wiki/xacro" name="husky">
-  <!-- robot name parameter -->
-  <!-- <xacro:arg name="name" default="" /> -->
   <xacro:arg name="prefix" default="" />
-  <xacro:arg name="gazebo_controllers" default="$(find clearpath_control)/config/control.yaml" />
-  <xacro:include filename="$(find clearpath_platform_description)/urdf/husky_macro.urdf.xacro" />
+  <xacro:arg name="gazebo_controllers" default="$(find clearpath_control)/config/a200/control.yaml" />
+  <xacro:include filename="$(find clearpath_platform_description)/urdf/a200/a200_macro.urdf.xacro" />
   <!-- Load husky description -->
-  <xacro:husky prefix="$(arg prefix)" />
+  <xacro:a200 prefix="$(arg prefix)" />
   <xacro:if value="$(arg is_sim)">
     <gazebo>

File: clearpath_platform_description/urdf/husky_macro.urdf.xacro (robot description, xacro)
@@ -20,5 +20,5 @@
   <xacro:include filename="$(find clearpath_platform_description)/urdf/accessories/sensor_arch.urdf.xacro"/>
   <xacro:property name="M_PI" value="3.14159"/>
-  <xacro:macro name="husky" params="prefix">
+  <xacro:macro name="a200" params="prefix">
     <!-- Base Size -->
     <xacro:property name="base_x_size" value="0.98740000" />
@@ -32,4 +32,5 @@
     <xacro:property name="wheel_length" value="0.1143" />
     <xacro:property name="wheel_radius" value="0.1651" />
+    <xacro:property name="wheel" value="" />
     <!-- Base link is the center of the robot's bottom plate -->
     <link name="${prefix}base_link">
@@ -90,16 +91,16 @@
     </joint>
     <!-- Husky wheel macros -->
-    <xacro:husky_wheel wheel_prefix="${prefix}front_left">
+    <xacro:wheel wheel_prefix="${prefix}front_left">
       <origin xyz="${wheelbase/2} ${track/2} ${wheel_vertical_offset}" rpy="0 0 0" />
-    </xacro:husky_wheel>
-    <xacro:husky_wheel wheel_prefix="${prefix}front_right">
+    </xacro:wheel>
+    <xacro:wheel wheel_prefix="${prefix}front_right">
       <origin xyz="${wheelbase/2} ${-track/2} ${wheel_vertical_offset}" rpy="0 0 0" />
-    </xacro:husky_wheel>
-    <xacro:husky_wheel wheel_prefix="${prefix}rear_left">
+    </xacro:wheel>
+    <xacro:wheel wheel_prefix="${prefix}rear_left">
       <origin xyz="${-wheelbase/2} ${track/2} ${wheel_vertical_offset}" rpy="0 0 0" />
-    </xacro:husky_wheel>
-    <xacro:husky_wheel wheel_prefix="${prefix}rear_right">
+    </xacro:wheel>
+    <xacro:wheel wheel_prefix="${prefix}rear_right">
       <origin xyz="${-wheelbase/2} ${-track/2} ${wheel_vertical_offset}" rpy="0 0 0" />
-    </xacro:husky_wheel>
+    </xacro:wheel>
     <xacro:husky_decorate />
     <!-- <xacro:if value="$(arg laser_enabled)">
